File: techin514_final_sensor_pcb/techin514_final_sensor_pcb.kicad_pcb (KiCad board)
At the start: 2 copper layers, 15 parts, among them J1 28BYJ-48 Stepper Motor, SW1 CK_KMS2xxGP, U1 ESP32-C3-DevKitM-1, U2 ESP32-C3-DevKitM-1, U3 ADXL343, U4 ULN2003, U5 TPS79301-EP

Commit message: update schematic and pcb
Parts:
- removed R5: R, Resistor_SMD:R_0603_1608Metric
- moved SW1 43.2 mm to (184.5, 93.4)
- moved BT2 33.5 mm to (150.5, 102.5)
- moved U4 9.08 mm to (139.5, 77.5)
- moved D1 8.00 mm to (140.6, 103.1)
- moved J1 2.00 mm to (151.0, 77.0)
Connections:
- SW1 pad SH: Net-(SW1-B) -> GND
- U2 pad 13: Net-(U2-5V-Pad13) -> /BATT(5V)
- U2 pad 14: Net-(U2-5V-Pad13) -> /BATT(5V)
- U2 pad 2: +3V3 -> Net-(U2-3V3-Pad2)
- U2 pad 3: +3V3 -> Net-(U2-3V3-Pad2)
Routing:
- net Net-(D1-DIN): track 0.00 -> 45.9 mm
- net /BATT(5V): track 0.00 -> 40.1 mm
- net Net-(U2-IO1): track 0.00 -> 35.8 mm
- net GND: track 0.00 -> 35.1 mm
- net Net-(U2-IO3): track 0.00 -> 28.3 mm
- net Net-(U2-IO0): track 0.00 -> 26.8 mm
- net Net-(U2-IO5): track 0.00 -> 9.22 mm
- net Net-(J1-Pin_4): track 0.00 -> 6.73 mm
- net Net-(J1-Pin_3): track 0.00 -> 5.36 mm
- net Net-(J1-Pin_2): track 0.00 -> 4.72 mm
- net Net-(J1-Pin_1): track 0.00 -> 4.09 mm

Commit message: update pcb
Parts:
- removed U3: ADXL343, Package_LGA:LGA-14_3x5mm_P0.8mm_LayoutBorder1x6y
- added U6: LSM6DS3, Package_LGA:LGA-14_3x2.5mm_P0.5mm_LayoutBorder3x4y, F.Cu at (57.0, 99.2)
- moved R4 8.83 mm to (62.3, 99.5)
- moved R3 3.28 mm to (57.1, 93.2)
Connections:
- R3 pad 1: +3V3 -> Net-(U1-IO0)
- R3 pad 2: Net-(U1-IO0) -> +3V3
- R4 pad 1: Net-(U3-~{CS}) -> Net-(U1-IO1)
Routing:
- net +3V3: track 63.1 -> 26.6 mm
- net GND: track 35.1 -> 46.1 mm
- net Net-(U1-IO1): track 21.7 -> 16.1 mm
- net Net-(U3-~{CS}): track 5.21 -> 0.00 mm
- net Net-(U1-IO0): track 25.4 -> 24.5 mm
- removed copper zone on B.Cu, net GND

Commit message: updated drl
Parts:
- moved U4 21.8 mm to (150.1, 96.5), turned to 180 degrees
- moved J1 20.9 mm to (137.0, 92.5), turned to -90 degrees
- moved R1 6.01 mm to (61.5, 73.3), turned to -90 degrees
- moved R3 4.46 mm to (61.5, 92.8), turned to 90 degrees
- moved R4 0.84 mm to (61.5, 99.3), turned to -90 degrees
- moved R2 0.53 mm to (57.5, 78.0), turned to 180 degrees
- turned SW1 to 90 degrees
Routing:
- net GND: track 46.1 -> 11.2 mm
- net Net-(U2-IO1): track 35.8 -> 6.58 mm
- net Net-(U2-IO2): track 0.00 -> 18.7 mm
- net Net-(U2-IO3): track 28.3 -> 12.5 mm
- net Net-(U2-IO0): track 26.8 -> 11.9 mm
- net Net-(J1-Pin_1): track 4.09 -> 10.4 mm
- net Net-(U1-IO0): track 24.5 -> 18.4 mm
- net Net-(U5-FB): track 12.3 -> 7.17 mm
- net +3V3: track 26.6 -> 31.7 mm
- net Net-(J1-Pin_4): track 6.73 -> 10.00 mm
- net /BATT(5V): track 40.1 -> 43.0 mm
- net Net-(J1-Pin_2): track 4.72 -> 7.46 mm
- net Net-(J1-Pin_3): track 5.36 -> 7.95 mm
- net Net-(U2-IO5): track 9.22 -> 11.5 mm
Other:
- board outline added: 141.5 x 76 mm

Commit message: updated schematic and PCB
Parts:
- removed BT1: Battery_Cell, Battery:BatteryHolder_Bulgin_BX0034_1xAAA
- removed BT2: Battery_Cell, Connector_PinHeader_1.00mm:PinHeader_1x02_P1.00mm_Vertical
- removed D1: WS2812, LED_SMD:LED_WS2812_PLCC6_5.0x5.0mm_P1.6mm
- removed R1, R2: R, Resistor_SMD:R_0603_1608Metric
- removed SW1: CK_KMS2xxGP, Button_Switch_SMD:SW_Push_1P1T-SH_NO_CK_KMR2xxG
- removed U4: ULN2003, Package_DIP:DIP-16_W7.62mm
- removed U5: TPS79301-EP, Package_SON:SON-8-1EP_3x2mm_P0.5mm_EP1.4x1.6mm
- removed U6: LSM6DS3, Package_LGA:LGA-14_3x2.5mm_P0.5mm_LayoutBorder3x4y
- added J10: J_PWR2, Connector_PinHeader_2.54mm:PinHeader_1x04_P2.54mm_Vertical, F.Cu at (182.5, 91.3)
- added J2: J_BAT, Connector_PinHeader_2.54mm:PinHeader_1x02_P2.54mm_Vertical, F.Cu at (83.7, 120.6)
- added J3: J_ULN_IN, Connector_PinHeader_2.54mm:PinHeader_1x04_P2.54mm_Vertical, F.Cu at (192.5, 91.4)
- added J4: J_LDO, Connector_PinHeader_2.54mm:PinHeader_1x02_P2.54mm_Vertical, F.Cu at (89.7, 122.9)
- added J5: J_MOTOR, Connector_PinHeader_2.54mm:PinHeader_1x05_P2.54mm_Vertical, F.Cu at (226.9, 92.2)
- added J6: J_IMU, Connector_PinHeader_2.54mm:PinHeader_1x04_P2.54mm_Vertical, F.Cu at (99.2, 95.1)
- added J7: J_PWR, Connector_PinHeader_2.54mm:PinHeader_1x02_P2.54mm_Vertical, F.Cu at (95.7, 119.8)
- added J8: J_LED, Connector_PinHeader_2.54mm:PinHeader_1x03_P2.54mm_Vertical, F.Cu at (221.4, 89.7)
- added J9: J_SW, Connector_PinHeader_2.54mm:PinHeader_1x02_P2.54mm_Vertical, F.Cu at (221.4, 104.2)
- J1: value 28BYJ-48 Stepper Motor -> J_BAT2; footprint Connector_PinHeader_1.00mm:PinHeader_1x05_P1.00mm_Vertical -> Connector_PinHeader_2.54mm:PinHeader_1x02_P2.54mm_Vertical
- R3, R4: footprint Resistor_SMD:R_0603_1608Metric -> Resistor_THT:R_Axial_DIN0207_L6.3mm_D2.5mm_P7.62mm_Horizontal
- U1, U2: value ESP32-C3-DevKitM-1 -> ~; footprint RF_Module:ESP32-C3-DevKitM-1 -> ESP32footprint:XIAO_ESP32
- moved J1 59.9 mm to (196.0, 82.0), turned to 0 degrees
- moved U2 59.6 mm to (206.9, 99.1)
- moved R4 46.6 mm to (106.5, 87.1)
- moved R3 38.5 mm to (99.2, 100.6), turned to -90 degrees
- moved U1 26.0 mm to (83.8, 94.3)
Connections:
- J1 pad 1: Net-(J1-Pin_1) -> Net-(J1-VBAT_5V)
- J1 pad 2: Net-(J1-Pin_2) -> Net-(J1-GND)
- R3 pad 1: Net-(U1-IO0) -> Net-(J6-SDA)
- R3 pad 2: +3V3 -> Net-(J4-3V3)
- R4 pad 1: Net-(U1-IO1) -> Net-(J6-SCL)
- R4 pad 2: +3V3 -> Net-(J4-3V3)
- U1 pad 1: GND -> unconnected-(U1-GPIO1_A0_D0-Pad1)
- U1 pad 10: Net-(U1-IO1) -> unconnected-(U1-GPIO8_A9_D9_CIPO-Pad10)
- U1 pad 12: GND -> Net-(J4-3V3)
- U1 pad 13: Net-(U1-5V-Pad13) -> Net-(J6-GND)
- U1 pad 14: Net-(U1-5V-Pad13) -> unconnected-(U1-5V-Pad14)
- U1 pad 15: GND -> Net-(J2-VBAT)
- U1 pad 16: GND -> Net-(J2-GND)
- U1 pad 2: +3V3 -> unconnected-(U1-GPIO2_A1_D1-Pad2)
- U1 pad 3: +3V3 -> unconnected-(U1-GPIO3_A2_D2-Pad3)
- U1 pad 5: unconnected-(U1-IO3-Pad5) -> Net-(J6-SDA)
- U1 pad 6: GND -> Net-(J6-SCL)
- U1 pad 8: GND -> unconnected-(U1-GPIO44_D7_RX-Pad8)
- U1 pad 9: Net-(U1-IO0) -> unconnected-(U1-GPIO7_A8_D8_SCK-Pad9)
- U2 pad 1: GND -> Net-(J1-VBAT_5V)
- U2 pad 11: unconnected-(U2-IO10-Pad11) -> Net-(J8-LED_DIN)
- U2 pad 12: GND -> unconnected-(U2-3V3-Pad12)
- U2 pad 13: /BATT(5V) -> unconnected-(U2-GND-Pad13)
- U2 pad 14: /BATT(5V) -> unconnected-(U2-5V-Pad14)
- U2 pad 15: GND -> unconnected-(U2-+BATT-Pad15)
- U2 pad 16: GND -> unconnected-(U2--BATT-Pad16)
- U2 pad 2: Net-(U2-3V3-Pad2) -> Net-(J1-GND)
- U2 pad 3: Net-(U2-3V3-Pad2) -> Net-(J3-MOTOR_IN3)
- U2 pad 5: Net-(U2-IO3) -> unconnected-(U2-GPIO4_A3_D3_SDA-Pad5)
- U2 pad 6: GND -> unconnected-(U2-GPIO6_A5_D5_SCL-Pad6)
- U2 pad 8: GND -> unconnected-(U2-GPIO44_D7_RX-Pad8)
Routing:
- net Net-(J6-GND): track 0.00 -> 68.7 mm
- net Net-(J6-SCL): track 0.00 -> 64.5 mm
- net Net-(D1-DIN): track 45.9 -> 0.00 mm
- net Net-(J4-3V3): track 0.00 -> 45.8 mm
- net /BATT(5V): track 43.0 -> 0.00 mm
- net Net-(J6-SDA): track 0.00 -> 40.6 mm
- net +3V3: track 31.7 -> 0.00 mm
- net Net-(J1-GND): track 0.00 -> 29.4 mm
- net Net-(J1-VBAT_5V): track 0.00 -> 29.2 mm
- net /BATT: track 21.4 -> 0.00 mm
- net Net-(U1-IO0): track 18.4 -> 0.00 mm
- net Net-(J3-MOTOR_IN3): track 0.00 -> 16.8 mm
- net Net-(U1-IO1): track 15.7 -> 0.00 mm
- net Net-(U2-IO3): track 12.5 -> 0.00 mm
- net Net-(J2-GND): track 0.00 -> 12.2 mm
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- added copper zone on F.Cu, net (none)
- removed copper zone on F.Cu, net GND
Other:
- board outline removed

Commit message: updated PCB
Parts:
- removed J1: J_BAT2, Connector_PinHeader_2.54mm:PinHeader_1x02_P2.54mm_Vertical
- removed J10: J_PWR2, Connector_PinHeader_2.54mm:PinHeader_1x04_P2.54mm_Vertical
- removed J3: J_ULN_IN, Connector_PinHeader_2.54mm:PinHeader_1x04_P2.54mm_Vertical
- removed J5: J_MOTOR, Connector_PinHeader_2.54mm:PinHeader_1x05_P2.54mm_Vertical
- removed J8: J_LED, Connector_PinHeader_2.54mm:PinHeader_1x03_P2.54mm_Vertical
- removed J9: J_SW, Connector_PinHeader_2.54mm:PinHeader_1x02_P2.54mm_Vertical
- removed U2: ~, ESP32footprint:XIAO_ESP32
- R3, R4: value R -> 4.7kOhm; footprint Resistor_THT:R_Axial_DIN0207_L6.3mm_D2.5mm_P7.62mm_Horizontal -> Resistor_SMD:R_0603_1608Metric
- moved J2 51.1 mm to (134.6, 115.8)
- moved J4 51.1 mm to (140.6, 118.1)
- moved J6 51.1 mm to (150.1, 90.3)
- moved J7 51.1 mm to (146.6, 115.1)
- moved R3 51.1 mm to (150.1, 95.8)
- moved U1 51.1 mm to (134.7, 89.5)
- moved R4 51.0 mm to (157.4, 83.7)
Routing:
- net Net-(J1-GND): track 29.4 -> 0.00 mm
- net Net-(J1-VBAT_5V): track 29.2 -> 0.00 mm
- net Net-(J3-MOTOR_IN3): track 16.8 -> 0.00 mm
- net Net-(J3-Pin_4): track 16.8 -> 0.00 mm
- net Net-(J8-LED_DIN): track 8.68 -> 0.00 mm
- net Net-(J9-Pin_2): track 7.12 -> 0.00 mm
- net Net-(J9-BTN): track 7.12 -> 0.00 mm
