File: techin514_final_sensor_pcb/techin514_final_sensor_pcb.kicad_pcb (KiCad board)
At the start: 2 copper layers, 7 parts, among them J2 J_BAT, J4 J_LDO, J6 J_IMU, J7 J_PWR

Commit message: update code
Routing:
- net Net-(J4-3V3): track 45.8 -> 113.8 mm
- net Net-(J2-VBAT): track 9.50 -> 20.9 mm
Other:
- board outline added: 39.5 x 50.5 mm
Changed lines of the file:
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@@
 	)
 	(gr_rect
-		(start 210.402161 109.1665)
-		(end 250.402161 159.1665)
+		(start 210 109)
+		(end 249.5 159.5)
 		(stroke
-			(width 0.2)
+			(width 0.05)
 			(type default)
 		)
 		(fill no)
-		(layer "F.Cu")
+		(layer "Edge.Cuts")
+	)
+	(segment
+		(start 221.963661 154.32505)
+		(end 221.963661 152.43)
+		(width 0.2)
+		(layer "F.Cu")
+		(net 1)
 	)
 	(segment
@@
 	)
 	(segment
+		(start 221.963661 152.43)
+		(end 223.064661 151.329)
+		(width 0.2)
+		(layer "F.Cu")
+		(net 1)
+	)
+	(segment
+		(start 227.698661 154.97)
+		(end 222.608611 154.97)
+		(width 0.2)
+		(layer "F.Cu")
+		(net 1)
+	)
+	(segment
 		(start 223.064661 145.219)
 		(end 220.669661 142.824)
@@
 	)
 	(segment
+		(start 222.608611 154.97)
+		(end 221.963661 154.32505)
+		(width 0.2)
+		(layer "F.Cu")
+		(net 1)
+	)
+	(segment
+		(start 229.064661 153.604)
+		(end 227.698661 154.97)
+		(width 0.2)
+		(layer "F.Cu")
+		(net 1)
+	)
+	(segment
 		(start 223.064661 153.869)
 		(end 225.749661 151.184)
@@
 	)
 	(segment
-		(start 245.902161 131.6115)
-		(end 238.564661 138.949)
+		(start 238.108611 117.108)
+		(end 245.778513 117.108)
 		(width 0.2)
 		(layer "F.Cu")
@@
 	)
 	(segment
+		(start 246.628161 117.957648)
+		(end 246.628161 119.274)
+		(width 0.2)
+		(layer "F.Cu")
+		(net 3)
+	)
+	(segment
+		(start 245.778513 117.108)
+		(end 246.628161 117.957648)
+		(width 0.2)
+		(layer "F.Cu")
+		(net 3)
+	)
+	(segment
+		(start 244.5 132)
+		(end 244.5 124.789289)
+		(width 0.2)
+		(layer "F.Cu")
+		(net 3)
+	)
+	(segment
+		(start 237.5 138)
+		(end 238 138.5)
+		(width 0.2)
+		(layer "F.Cu")
+		(net 3)
+	)
+	(segment
 		(start 235.239661 122.504)
 		(end 238.564661 125.829)
@@
 	)
 	(segment
-		(start 237.513661 137.898)
-		(end 237.513661 126.88)
-		(width 0.2)
-		(layer "F.Cu")
-		(net 3)
-	)
-	(segment
-		(start 238.564661 138.949)
-		(end 237.513661 137.898)
+		(start 229.064661 151.064)
+		(end 247.304161 132.8245)
+		(width 0.2)
+		(layer "F.Cu")
+		(net 3)
+	)
+	(segment
+		(start 247.304161 121.402)
+		(end 245.902161 120)
+		(width 0.2)
+		(layer "F.Cu")
+		(net 3)
+	)
+	(segment
+		(start 238.108611 119.31)
+		(end 237.463661 118.66505)
+		(width 0.2)
+		(layer "F.Cu")
+		(net 3)
+	)
+	(segment
+		(start 247.304161 132.8245)
+		(end 247.304161 121.402)
+		(width 0.2)
+		(layer "F.Cu")
+		(net 3)
+	)
+	(segment
+		(start 238 138.5)
+		(end 244.5 132)
+		(width 0.2)
+		(layer "F.Cu")
+		(net 3)
+	)
+	(segment
+		(start 239.020711 119.31)
+		(end 238.108611 119.31)
+		(width 0.2)
+		(layer "F.Cu")
+		(net 3)
+	)
+	(segment
+		(start 237.463661 118.66505)
+		(end 237.463661 117.75295)
+		(width 0.2)
+		(layer "F.Cu")
+		(net 3)
+	)
+	(segment
+		(start 237.838661 126.555)
+		(end 238.564661 125.829)
 		(width 0.2)
 		(layer "F.Cu")
@@
 	)
 	(segment
+		(start 246.628161 119.274)
+		(end 245.902161 120)
+		(width 0.2)
+		(layer "F.Cu")
+		(net 3)
+	)
+	(segment
+		(start 238.564661 125.829)
+		(end 237.5 126.893661)
+		(width 0.2)
+		(layer "F.Cu")
+		(net 3)
+	)
+	(segment
 		(start 234.554661 151.064)
 		(end 235.064661 150.554)
@@
 	)
 	(segment
-		(start 237.513661 126.88)
-		(end 238.564661 125.829)
-		(width 0.2)
-		(layer "F.Cu")
-		(net 3)
-	)
-	(segment
-		(start 245.902161 125.4765)
-		(end 245.902161 131.6115)
+		(start 244.5 124.789289)
+		(end 239.020711 119.31)
+		(width 0.2)
+		(layer "F.Cu")
+		(net 3)
+	)
+	(segment
+		(start 238.564661 132.154)
+		(end 237.838661 131.428)
+		(width 0.2)
+		(layer "F.Cu")
+		(net 3)
+	)
+	(segment
+		(start 237.838661 131.428)
+		(end 237.838661 126.555)
+		(width 0.2)
+		(layer "F.Cu")
+		(net 3)
+	)
+	(segment
+		(start 237.463661 117.75295)
+		(end 238.108611 117.108)
+		(width 0.2)
+		(layer "F.Cu")
+		(net 3)
+	)
+	(segment
+		(start 237.5 126.893661)
+		(end 237.5 138)
 		(width 0.2)
 		(layer "F.Cu")
@@
 	)
 	(segment
-		(start 241.064661 123.249)
-		(end 238.564661 120.749)
+		(start 238.564661 130.504)
+		(end 239.496 130.504)
 		(width 0.2)
 		(layer "F.Cu")
@@
 	)
 	(segment
+		(start 241 122.5)
+		(end 240.315661 122.5)
+		(width 0.2)
+		(layer "F.Cu")
+		(net 6)
+	)
+	(segment
 		(start 215.224661 127.949)
 		(end 215.589661 127.584)
@@
 	)
 	(segment
-		(start 241.064661 128.829)
-		(end 241.064661 123.249)
+		(start 240.315661 122.5)
+		(end 238.564661 120.749)
+		(width 0.2)
+		(layer "F.Cu")
+		(net 6)
+	)
+	(segment
+		(start 241 129)
+		(end 241 122.5)
+		(width 0.2)
+		(layer "F.Cu")
+		(net 6)
+	)
+	(segment
+		(start 239.496 130.504)
+		(end 241 129)
 		(width 0.2)
 		(layer "F.Cu")
@@
 		(start 236.639661 118.824)
 		(end 224.349661 118.824)
-		(width 0.2)
-		(layer "F.Cu")
-		(net 6)
-	)
-	(segment
-		(start 238.564661 131.329)
-		(end 241.064661 128.829)
 		(width 0.2)
 		(layer "F.Cu")
@@
 		(polygon
 			(pts
-				(xy 210.402161 109.1665) (xy 250.402161 109.1665) (xy 250.402161 159.1665) (xy 210.402161 159.1665)
+				(xy 210 109) (xy 249.5 109) (xy 249.5 159.5) (xy 210 159.5)
 			)
 		)
