File: hardware/pcb/sensor_tag/C3_GestureDriver.kicad_pcb (KiCad board)
At the start: 2 copper layers, 37 x 32.5 mm, 17 parts, among them J1 BAT, J2 USART, SW2 SW_SPDT, U1 XIAO_ESP32, U2 LSM6DS3, U3 MCP1700-3302E_TO

Commit message: update
Parts:
- removed the U2 at (90.5, 146.0)
- U2: moved to B.Cu
- moved C2 11.5 mm to (83.0, 137.0)
- moved R3 9.50 mm to (83.0, 148.0)
- moved L1 5.50 mm to (83.0, 146.0), turned to 180 degrees
- moved U2 4.50 mm to (83.0, 141.0), turned to -90 degrees
- moved C1 1.50 mm to (83.0, 144.0)
- moved J2 0.23 mm to (57.0, 121.0)
- turned C3 to 0 degrees
Routing:
- net /TX: track 33.5 -> 74.0 mm
- net +3.3V: track 52.6 -> 55.1 mm
- net /LSM6DS3_SCL: track 21.0 -> 18.9 mm
- net /LSM6DS3_SDA: track 24.0 -> 21.9 mm
- net Net-(U2-CS): track 8.18 -> 9.90 mm
- net Net-(U2-VDD): track 3.85 -> 4.50 mm
- added copper zone on B.Cu, net GND

Commit message: update everything
Routing:
- net Net-(J1-Pin_2): track 7.93 -> 8.74 mm
- net /LSM6DS3_SCL: track 18.9 -> 18.3 mm
Other:
- board size 37 x 32.5 mm -> 38.5 x 33.5 mm
